Commit message: fixed bug in contactimplicit on gravity in dynamics

File: systems/urdf/sliding_block.urdf (robot description, URDF)
Before this commit: robot sliding_block, 4 links, 3 joints
Links:
- link box: geometry collision sphere radius=0; visual box size=1 1 1

Commit message: Updated contact_implicit_test to test constraint values

File: systems/urdf/sliding_block.urdf (robot description, URDF)
Before this commit: robot sliding_block, 4 links, 3 joints
Links:
- removed link yrot
Joints:
- removed joint yspin
- joint zslide: child yrot -> box
