Commit message: warning 31, iteration limit reached for hopper example

File: systems/urdf/single_legged_hopper.urdf (robot description, URDF)
Before this commit: robot single_legged_hopper, 6 links, 5 joints
Joints:
- joint base_leg_1: limit lower=-0.785 upper=0.785 effort=1000 velocity=1 -> lower=-0.785 upper=0.785
- joint leg_1_leg_2: limit lower=-0.785 upper=0.785 effort=1000 velocity=1 -> lower=-1.5 upper=1.5
- joint leg_2_foot: limit lower=-0.785 upper=0.785 effort=1000 velocity=1 -> lower=-0.785 upper=0.785

Commit message: pre updating contactimplicity class

File: systems/urdf/single_legged_hopper.urdf (robot description, URDF)
Before this commit: robot single_legged_hopper, 6 links, 5 joints
Links:
- link foot: geometry collision sphere radius=0; visual box size=0.3 0.01 0.01

Commit message: solveing hopper

File: systems/urdf/single_legged_hopper.urdf (robot description, URDF)
Before this commit: robot single_legged_hopper, 6 links, 5 joints
Links:
- link foot: geometry collision sphere radius=0; collision sphere radius=0
Joints:
- joint base_leg_1: limit lower=-0.785 upper=0.785 -> lower=-1.57 upper=1.57
- joint leg_1_leg_2: limit lower=-1.5 upper=1.5 -> lower=-1.04 upper=2.09
- joint leg_2_foot: limit lower=-0.785 upper=0.785 -> lower=-1.04 upper=1.04

Commit message: hopper

File: systems/urdf/single_legged_hopper.urdf (robot description, URDF)
Before this commit: robot single_legged_hopper, 6 links, 5 joints
Links:
- link base: mass 1 -> 10
- link foot: mass 0.3 -> 0.33; geometry collision sphere radius=0; collision sphere radius=0

Commit message: branch for IEEE Access

File: systems/urdf/single_legged_hopper.urdf (robot description, URDF)
Before this commit: robot single_legged_hopper, 6 links, 5 joints
Links:
- link foot: geometry collision sphere radius=0; collision sphere radius=0
